Commit message: New URDF

File: Assets/my-robot/robot.urdf (robot description, URDF)
Before this commit: robot my-robot, 11 links, 10 joints
Links:
- link cushion_left: geometry collision mesh filename=package://assets/cushion_left.stl; visual mesh filename=package://assets/cushion_left.stl
- link cushion_right: geometry collision mesh filename=package://assets/cushion_right.stl; visual mesh filename=package://assets/cushion_right.stl

File: Assets/my-robot/robot_simplified.urdf (robot description, URDF)
Before this commit: robot my-robot, 11 links, 10 joints
Links:
- link cushion_left: geometry collision mesh filename=package://assets/cushion_left.stl; visual mesh filename=package://assets/cushion_left.stl
- link cushion_right: geometry collision mesh filename=package://assets/cushion_right.stl; visual mesh filename=package://assets/cushion_right.stl
